File: data_logger_wsu_racing_v0.3.kicad_pro.kicad_sch (KiCad schematic)
At the start: 41 parts, among them J1 DB15_Female_MountingHoles, J2 USB_B, U1 LM2592HV, U2 ADXL362_BOB, U3 MCP2562, U4 Teensy4.1

Commit message: Fixed D+ and D- lines on the USB host bus.
Connections:
- net D+: now also J2.3 (D+); no longer J2.2 (D-)
- net D-: now also J2.2 (D-); no longer J2.3 (D+)
Changed lines of the file:
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@@
-    (stroke (width 0) (type default) (color 0 0 0 0))
-  )
-  (wire (pts (xy 231.14 48.26) (xy 251.46 48.26))
     (stroke (width 0) (type default) (color 0 0 0 0))
   )
@@
     (stroke (width 0) (type default) (color 0 0 0 0))
   )
+  (wire (pts (xy 231.14 48.26) (xy 234.95 48.26))
+    (stroke (width 0) (type default) (color 0 0 0 0))
+  )
   (wire (pts (xy 40.64 168.91) (xy 40.64 170.18))
     (stroke (width 0) (type default) (color 0 0 0 0))
@@
     (stroke (width 0) (type default) (color 0 0 0 0))
   )
-  (wire (pts (xy 231.14 50.8) (xy 251.46 50.8))
-    (stroke (width 0) (type default) (color 0 0 0 0))
-  )
   (polyline (pts (xy 17.78 120.65) (xy 99.06 120.65))
     (stroke (width 0) (type default) (color 0 0 0 0))
@@
     (stroke (width 0) (type default) (color 0 0 0 0))
   )
+  (wire (pts (xy 231.14 50.8) (xy 234.95 50.8))
+    (stroke (width 0) (type default) (color 0 0 0 0))
+  )
   (wire (pts (xy 123.19 49.53) (xy 121.92 49.53))
     (stroke (width 0) (type default) (color 0 0 0 0))
@@
     (stroke (width 0) (type default) (color 0 0 0 0))
   )
+  (wire (pts (xy 247.65 50.8) (xy 251.46 50.8))
+    (stroke (width 0) (type default) (color 0 0 0 0))
+  )
   (wire (pts (xy 134.62 132.08) (xy 134.62 130.81))
     (stroke (width 0) (type default) (color 0 0 0 0))
@@
   )
   (wire (pts (xy 57.15 162.56) (xy 67.31 162.56))
+    (stroke (width 0) (type default) (color 0 0 0 0))
+  )
+  (wire (pts (xy 247.65 48.26) (xy 251.46 48.26))
     (stroke (width 0) (type default) (color 0 0 0 0))
   )
@@
     (effects (font (size 1.27 1.27)) (justify left bottom))
   )
+  (label "D+" (at 247.65 50.8 0)
+    (effects (font (size 1.27 1.27)) (justify left bottom))
+  )
   (label "car_A3" (at 66.04 129.54 0)
     (effects (font (size 1.27 1.27)) (justify left bottom))
@@
     (effects (font (size 0.9906 0.9906)) (justify right bottom))
   )
+  (label "D-" (at 247.65 48.26 0)
+    (effects (font (size 1.27 1.27)) (justify left bottom))
+  )
   (label "teensy_A3" (at 82.55 137.16 180)
